Commit message: update. simpler directory
follow

File: farm_ws/src/farm_description/urdf/ugvbeast_arm.urdf (robot description, URDF)
Before this commit: robot turtlebot3_waffle_for_open_manipulator, 20 links, 19 joints
Links:
- removed link caster_back_left_link
- removed link caster_back_right_link
- link base_link: geometry collision box size=0.24 0.2 0.12; visual mesh filename=../../meshes/ugv_beast/base_link.stl scale=1.0 1.0 1.0
- link base_scan: geometry collision cylinder length=0.0315 radius=0.045; visual mesh filename=../../meshes/ugv_beast/base_lidar_link.stl scale=1.0 1.0 1.0
- link camera_link: geometry collision box size=0.02 0.09 0.03; visual mesh filename=../../meshes/ugv_beast/3d_camera_link.stl scale=1.0 1.0 1.0
- link wheel_left_link: mass 2.8498940e-02 -> 0.1; geometry collision cylinder length=0.03 radius=0.04
- link wheel_right_link: mass 2.8498940e-02 -> 0.1; geometry collision cylinder length=0.03 radius=0.04
Joints:
- removed joint caster_back_left_joint
- removed joint caster_back_right_joint
- joint arm_base_joint: origin xyz=0.0 0.0 0.12 rpy=0 0 0 -> xyz=-0.04 0.0 0.12 rpy=0 0 3.14159
- joint base_joint: origin xyz=0 0 0.010 rpy=0 0 0 -> xyz=0 0 0.021 rpy=0 0 0
- joint camera_depth_joint: origin xyz=0.005 0.027999999999999997 0.013 rpy=0 0 0 -> xyz=0.01 0 0 rpy=0 0 0
- joint camera_joint: origin xyz=0.064 -0.065 0.094 rpy=0 0 0 -> xyz=0.07 0 0.098 rpy=0 0 0
- joint camera_rgb_joint: origin xyz=0.005 0.018 0.013 rpy=0 0 0 -> xyz=0 0 0 rpy=0 0 0
- joint scan_joint: origin xyz=-0.024 0 0.122 rpy=0 0 0 -> xyz=0.05 0 0.11 rpy=0 0 0
- joint wheel_left_joint: origin xyz=0.0 0.144 0.023 rpy=-1.57 0 0 -> xyz=0.0 0.09 0.02 rpy=-1.57 0 0
- joint wheel_right_joint: origin xyz=0.0 -0.144 0.023 rpy=-1.57 0 0 -> xyz=0.0 -0.09 0.02 rpy=-1.57 0 0
